File: HandymanSchematic_G0/Digital.kicad_sch (KiCad schematic)
At the start: 36 parts, among them J1 SWD Header, J2 PWR, J3 JACKS, J4 FOOTSWITCH, J5 ScopeGroundLoop, Q3 2N7002, Q4 2N7002, SW1 RST, SW2 BYP, U4 STM32G030F6P6, U5 AMS1117, U6 SSD1306

Commit message: board outline for 1590B size
Parts:
- U6: footprint Display:SSD1306_OLED_128x64 -> Display:SSD1306_OLED_128x64_OffBoard
Changed lines of the file:
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@@
 	(label "SCL"
 		(at 265.43 55.88 180)
-		(fields_autoplaced yes)
 		(effects
 			(font
@@
 	(label "SCL"
 		(at 59.69 73.66 180)
-		(fields_autoplaced yes)
 		(effects
 			(font
@@
 	(label "TunerModeIn"
 		(at 106.68 60.96 0)
-		(fields_autoplaced yes)
 		(effects
 			(font
@@
 	(label "GateByp"
 		(at 125.73 76.2 0)
-		(fields_autoplaced yes)
 		(effects
 			(font
@@
 	(label "SDA"
 		(at 59.69 76.2 180)
-		(fields_autoplaced yes)
 		(effects
 			(font
@@
 	(label "SDA"
 		(at 255.27 52.07 180)
-		(fields_autoplaced yes)
 		(effects
 			(font
@@
 	(label "GateLED"
 		(at 101.6 73.66 0)
-		(fields_autoplaced yes)
 		(effects
 			(font
@@
 	(label "TunerModeIn"
 		(at 200.66 101.6 0)
-		(fields_autoplaced yes)
 		(effects
 			(font
@@
 	(label "GateLED"
 		(at 195.58 60.96 180)
-		(fields_autoplaced yes)
 		(effects
 			(font
@@
 			)
 		)
-		(property "Footprint" "Display:SSD1306_OLED_128x64"
+		(property "Footprint" "Display:SSD1306_OLED_128x64_OffBoard"
 			(at 233.68 30.48 0)
 			(effects

Commit message: prelim layout
Parts:
- removed C17: 100n, Capacitor_SMD:C_0805_2012Metric, symbol Device:C
- removed C20: 10u, Capacitor_THT:CP_Radial_D5.0mm_P2.50mm, symbol Device:C_Polarized_US
- removed C23: 4u7, Capacitor_THT:CP_Radial_D5.0mm_P2.50mm, symbol Device:C_Polarized_US
- removed TP6: In, TestPoint:TestPoint_THTPad_D2.0mm_Drill1.0mm_VAL, symbol Connector:TestPoint
- removed TP7: Out, TestPoint:TestPoint_THTPad_D2.0mm_Drill1.0mm_VAL, symbol Connector:TestPoint
- removed TP9: OI, TestPoint:TestPoint_THTPad_D2.0mm_Drill1.0mm_VAL, symbol Connector:TestPoint
- added C13: 10u, Capacitor_SMD:C_0805_2012Metric, symbol Device:C
- renumbered C19 to C14, C21 to C16, C22 to C17, C24 to C19, C25 to C20, D10 to D8, D11 to D9, Q3 to Q2, Q4 to Q3, TP10 to TP7, TP11 to TP8, U4 to U3, U5 to U4, U6 to U5
Connections:
- net +3.3V: now also C13.2
- net FX_IN: now also J4.2 (Pin_2); no longer J4.1 (Pin_1)
- net FX_OUT: now also J4.1 (Pin_1); no longer J4.2 (Pin_2)
- net GND: now also C13.1
Other:
- moved on the sheet: C14, C17, TP7

Commit message: routed, DRC passing
Connections:
- net FX_IN: now also J4.1 (Pin_1); no longer J4.2 (Pin_2)
- net FX_OUT: now also J4.2 (Pin_2); no longer J4.1 (Pin_1)
Changed lines of the file:
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@@
 	(global_label "FX_IN"
 		(shape input)
-		(at 191.77 99.06 0)
+		(at 193.04 96.52 0)
 		(fields_autoplaced yes)
 		(effects
@@
 		)
 		(property "Intersheetrefs" "${INTERSHEET_REFS}"
-			(at 199.9562 99.06 0)
+			(at 201.2262 96.52 0)
 			(effects
 				(font
@@
 	(global_label "FX_OUT"
 		(shape output)
-		(at 193.04 96.52 0)
+		(at 191.77 99.06 0)
 		(fields_autoplaced yes)
 		(effects
@@
 		)
 		(property "Intersheetrefs" "${INTERSHEET_REFS}"
-			(at 202.9195 96.52 0)
+			(at 201.6495 99.06 0)
 			(effects
 				(font
