File: HandymanSchematic_G0/HandymanSchematic_G0.kicad_pcb (KiCad board)
At the start: 4 copper layers, 86 x 54 mm, 103 parts, among them J1 SWD Header, J2 PWR, J3 JACKS, J4 FOOTSWITCH, J5 ScopeGroundLoop, Q1 BC847, Q2 BC847, Q3 2N7002, Q4 2N7002, SW1 RST, SW2 BYP, U1 TL074, U2 TL074, U3 TL072, U4 STM32G030F6P6, U5 AMS1117, U6 SSD1306, Y1 32.768kHZ

Commit message: board outline for 1590B size
Parts:
- removed C16, C18: 6p, Capacitor_SMD:C_0805_2012Metric
- removed D8, D9: PMEG3030, Diode_SMD:D_SOD-123
- removed TP1: AK, TestPoint:TestPoint_THTPad_D2.0mm_Drill1.0mm_VAL
- removed TP2: AA, TestPoint:TestPoint_THTPad_D2.0mm_Drill1.0mm_VAL
- removed Y1: 32.768kHZ, Crystal:Crystal_SMD_SeikoEpson_MC306-4Pin_8.0x3.2mm
- C11, C2, C3, C7, C8, D4, D5, D6, D7, Q1, Q2, R10, R11, R12, R14, R18, R19, R2, R20, R21, R4, R6, R9, U2: moved to B.Cu
- C17, C19, C20, C21, C22, C23, C24, C25, J5, R29, R30, R31, R36, R37, SW1, TP10, TP11, TP6, TP7, TP9, U4, U5: moved to F.Cu
- U6: footprint Display:SSD1306_OLED_128x64 -> Display:SSD1306_OLED_128x64_OffBoard
- moved D1 261.6 mm to (-194.6, 1.80), turned to -90 degrees
- moved U1 261.4 mm to (-199.8, 5.40), turned to 180 degrees
- moved D2 259.5 mm to (-192.1, 1.80), turned to 90 degrees
- moved C4 257.0 mm to (-194.2, 5.38), turned to 0 degrees
- moved R3 253.7 mm to (-189.8, 2.38)
- moved R8 249.9 mm to (-194.2, 8.72), turned to 180 degrees
- moved R7 248.5 mm to (-190.6, 8.75), turned to 180 degrees
- moved R1 248.4 mm to (-187.6, 2.35)
- moved C5 247.3 mm to (-192.3, 10.8), turned to 0 degrees
- moved TP5 241.9 mm to (-160.0, -23.8)
- moved D6 241.1 mm to (-155.3, -22.3)
- moved TP7 236.4 mm to (-165.6, 46.4), turned to 0 degrees
- moved C24 235.6 mm to (-171.9, 57.1)
- moved D7 235.4 mm to (-155.3, -18.9)
- moved U2 235.4 mm to (-159.8, -10.0), turned to 180 degrees
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Connections:
- C21 pad 2: VCC -> +9V
- J1 pad 1: Net-(D8-A) -> +3.3V
- R16 pad 2: Net-(R16-Pad2) -> /Analog/Thresh
- R17 pad 1: /Analog/Thresh -> Net-(R17-Pad1)
- RV2 pad 1: Net-(R16-Pad2) -> /Analog/Thresh
- RV2 pad 2: /Analog/Thresh -> Net-(R17-Pad1)
- RV2 pad 3: /Analog/Thresh -> Net-(R17-Pad1)
- U4 pad 2: Net-(U4-PC14/PB9) -> unconnected-(U4-PC14/PB9-Pad2)
- U4 pad 3: Net-(U4-PC15) -> unconnected-(U4-PC15-Pad3)
- U5 pad 3: VCC -> +9V
Routing:
- net +3.3V: track 167.8 -> 0.00 mm, vias 3 -> 0
- net +9V: track 153.7 -> 0.00 mm, vias 6 -> 0
- net /Analog/VG: track 130.2 -> 0.00 mm, vias 5 -> 0
- net VCC: track 63.9 -> 0.00 mm, vias 2 -> 0
- net OPEN_IN: track 63.5 -> 0.00 mm, vias 1 -> 0
- net CLOSED_OUT: track 56.3 -> 0.00 mm
- net /Analog/SumPt: track 55.6 -> 0.00 mm, vias 2 -> 0
- net LOOP_OUT: track 48.9 -> 0.00 mm, vias 1 -> 0
- net GND: track 43.2 -> 0.00 mm, vias 201 -> 0
- net /Digital/TunerModeIn: track 43.2 -> 0.00 mm, vias 2 -> 0
- net FX_IN: track 42.7 -> 0.00 mm
- net LOOP_IN: track 32.1 -> 0.00 mm, vias 1 -> 0
- net /Analog/Thresh: track 31.4 -> 0.00 mm
- net SWDIO: track 28.8 -> 0.00 mm
- net SWCLK: track 28.2 -> 0.00 mm
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- removed copper zone on B.Cu, net GND
- removed copper zone on F.Cu, net GND
Other:
- board size 86 x 54 mm -> 55.7 x 44.8 mm
- board text removed: "Handyman v1"
- board text removed: "Rev. 1 - Feb 2025 Hayden Setlik"

Commit message: analog tweaks, 2 fewer op amps
Parts:
- C2, C8, Q1, Q2, R2, R4, R6: moved to F.Cu
- R31: moved to B.Cu
- moved D4 190.3 mm to (-95.3, 151.6), turned to 90 degrees
- moved D6 183.2 mm to (-97.9, 151.7), turned to 90 degrees
- moved D5 182.5 mm to (-95.3, 146.7), turned to 90 degrees
- moved D3 179.6 mm to (-135.6, 146.2), turned to 0 degrees
- moved C7 176.1 mm to (-107.1, 159.1)
- moved D7 175.4 mm to (-97.9, 146.8), turned to 90 degrees
- moved J3 174.1 mm to (-114.0, 164.2)
- moved R17 172.1 mm to (-138.5, 157.9), turned to 90 degrees
- moved R9 171.6 mm to (-107.1, 157.0), turned to 0 degrees
- moved R10 170.4 mm to (-101.2, 158.2)
- moved U2 169.6 mm to (-104.1, 150.1), turned to 90 degrees
- moved C8 168.1 mm to (-115.0, 155.4), turned to 0 degrees
- moved C3 166.5 mm to (-104.1, 155.7), turned to -90 degrees
- moved C1 165.8 mm to (-117.3, 150.9)
- moved R11 163.7 mm to (-107.0, 155.0)
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
Commit message: prelim layout
Parts:
- removed C15: 10n, Capacitor_SMD:C_0805_2012Metric
- removed C21, C22, C25: 100n, Capacitor_SMD:C_0805_2012Metric
- removed C23: 4u7, Capacitor_THT:CP_Radial_D5.0mm_P2.50mm
- removed C24: 220u, Capacitor_THT:CP_Radial_D5.0mm_P2.50mm
- removed D10: Orange, LED_THT:LED_D3.0mm
- removed D11: Green, LED_THT:LED_D3.0mm
- removed Q4: 2N7002, Package_TO_SOT_SMD:SOT-23
- removed TP10: TI, TestPoint:TestPoint_THTPad_D2.0mm_Drill1.0mm_VAL
- removed TP11: CO, TestPoint:TestPoint_THTPad_D2.0mm_Drill1.0mm_VAL
- removed TP4: VG, TestPoint:TestPoint_THTPad_D2.0mm_Drill1.0mm_VAL
- removed TP5: Env, TestPoint:TestPoint_THTPad_D2.0mm_Drill1.0mm_VAL
- removed TP6: In, TestPoint:TestPoint_THTPad_D2.0mm_Drill1.0mm_VAL
- removed TP9: OI, TestPoint:TestPoint_THTPad_D2.0mm_Drill1.0mm_VAL
- removed U6: SSD1306, Display:SSD1306_OLED_128x64_OffBoard
- added C16: 100n, Capacitor_SMD:C_0805_2012Metric, F.Cu at (44.8, 2.09)
- added D8: Orange, LED_THT:LED_D3.0mm, F.Cu at (2.05, 12.2)
- added D9: Green, LED_THT:LED_D3.0mm, F.Cu at (10.9, 12.1)
- added TP1: Thr, TestPoint:TestPoint_THTPad_D2.0mm_Drill1.0mm_VAL, B.Cu at (2.23, 36.1)
- added TP8: CO, TestPoint:TestPoint_THTPad_D2.0mm_Drill1.0mm_VAL, F.Cu at (33.8, 19.0)
- C10: value 100n -> 1u
- C12: value 22n -> 10n
- C13: value 1u -> 10u; moved to F.Cu
- C14, J1: moved to F.Cu
- C19: value 100n -> 220u; footprint Capacitor_SMD:C_0805_2012Metric -> Capacitor_THT:CP_Radial_D5.0mm_P2.50mm; moved to B.Cu
- C2: value 100n -> 10n; moved to B.Cu
- C20: value 10u -> 100n; footprint Capacitor_THT:CP_Radial_D5.0mm_P2.50mm -> Capacitor_SMD:C_0805_2012Metric; moved to B.Cu
- C5: value 10n -> 100n
- C6: value 33n -> 1u
- C8: value 33n -> 100n; moved to B.Cu
- C9: value 1u -> 22n
- Q1, R29, SW1: moved to B.Cu
- Q2: value BC847 -> 2N7002
- R1, R12, R21, R24: value 100k -> 470k
- R10: value 220k -> 47k
- R11: value 470k -> 1k
- R13: value 1k -> 470k
- R14: value 51k -> 5k6
- R15: value 5k6 -> 51k
- R2: value 10k -> 470k; moved to B.Cu
- R20: value 470k -> 180k
- R22: value 180k -> 100k
- R25: value 220k -> 470k
- R3: value 100k -> 10k
- R4, R6: value 47k -> 100k; moved to B.Cu
- R5: value 100k -> 47k
- R7: value 470k -> 47k
- R9: value 470k -> 100k
- TP3: value Thr -> Env
- TP7: value Out -> TI
- U3: value TL072 -> STM32G030F6P6; footprint Package_SO:SOIC-8_3.9x4.9mm_P1.27mm -> Package_SO:TSSOP-20_4.4x6.5mm_P0.65mm; moved to F.Cu
- U4: value STM32G030F6P6 -> AMS1117; footprint Package_SO:TSSOP-20_4.4x6.5mm_P0.65mm -> Package_TO_SOT_SMD:SOT-223-3_TabPin2
- U5: value AMS1117 -> SSD1306; footprint Package_TO_SOT_SMD:SOT-223-3_TabPin2 -> Display:SSD1306_OLED_128x64_OffBoard
- moved R29 248.3 mm to (45.0, 10.2), turned to -90 degrees
- moved SW1 235.9 mm to (44.8, 14.8), turned to -90 degrees
- moved J5 224.0 mm to (18.5, 6.44), turned to -90 degrees
- moved C10 220.1 mm to (47.3, 32.4), turned to 90 degrees
- moved U5 219.3 mm to (27.7, 2.58), turned to 180 degrees
- moved Q3 218.9 mm to (11.4, 16.2), turned to 180 degrees
- moved R34 214.4 mm to (14.4, 16.2), turned to -90 degrees
- moved R13 213.1 mm to (37.7, 23.4), turned to 180 degrees
- moved R35 211.7 mm to (16.4, 12.1), turned to 180 degrees
- moved R22 211.1 mm to (44.5, 33.1), turned to 0 degrees
- moved C19 210.6 mm to (47.6, 4.49), turned to -90 degrees
- moved R7 209.8 mm to (41.2, 19.1)
- moved C17 209.4 mm to (44.8, 5.97), turned to 180 degrees
- moved R33 208.3 mm to (7.62, 12.3), turned to 180 degrees
- moved R15 205.4 mm to (34.6, 37.4), turned to 180 degrees
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Connections:
- C1 pad 1: FX_IN -> +9V
- C1 pad 2: Net-(C1-Pad2) -> GND
- C10 pad 1: /Analog/Thresh -> Net-(C10-Pad1)
- C10 pad 2: GND -> LOOP_OUT
- C11 pad 1: Net-(C11-Pad1) -> FX_IN
- C11 pad 2: LOOP_OUT -> Net-(C11-Pad2)
- C12 pad 1: OPEN_IN -> /Analog/VG
- C12 pad 2: GND -> Net-(U1C--)
- C13 pad 1: FX_IN -> GND
- C13 pad 2: Net-(C13-Pad2) -> +3.3V
- C14 pad 1: +9V -> GND
- C14 pad 2: GND -> +3.3V
- C17 pad 2: NRST -> +3.3V
- C19 pad 1: GND -> +9V
- C19 pad 2: +3.3V -> GND
- C2 pad 1: Net-(Q1-B) -> Net-(U1B-+)
- C20 pad 1: +3.3V -> GND
- C20 pad 2: GND -> +3.3V
- C4 pad 1: +9V -> Net-(Q1-B)
- C5 pad 1: Net-(U1B-+) -> FX_IN
- C5 pad 2: GND -> Net-(C5-Pad2)
- C6 pad 1: Net-(U1D-+) -> LOOP_IN
- C6 pad 2: /Analog/VG -> Net-(C6-Pad2)
- C7 pad 1: LOOP_IN -> /Analog/Env
- C7 pad 2: Net-(C7-Pad2) -> /Analog/VG
- C8 pad 1: Net-(Q2-C) -> /Analog/Thresh
- C9 pad 1: /Analog/Env -> OPEN_IN
- C9 pad 2: /Analog/VG -> GND
- D2 pad 1: /Analog/HalfRect -> Net-(D2-K)
- D2 pad 2: Net-(D1-K) -> Net-(D2-A)
- D3 pad 1: Net-(D3-K) -> /Analog/HalfRect
- D3 pad 2: Net-(D3-A) -> Net-(D2-K)
- J4 pad 1: FX_IN -> FX_OUT
- J4 pad 2: FX_OUT -> FX_IN
- Q1 pad 3: Net-(Q1-C) -> Net-(D1-A)
- Q2 pad 1: Net-(Q1-C) -> CLOSED_OUT
- Q2 pad 2: /Analog/VG -> GND
- Q2 pad 3: Net-(Q2-C) -> Net-(D8-K)
- Q3 pad 1: CLOSED_OUT -> /Digital/GateLED
- R1 pad 1: Net-(C1-Pad2) -> +9V
- R1 pad 2: Net-(D1-A) -> Net-(U1B-+)
- R10 pad 1: Net-(Q2-C) -> Net-(R10-Pad1)
- R11 pad 1: Net-(U2B--) -> /Analog/HalfRect
- R11 pad 2: Net-(R11-Pad2) -> /Analog/Env
- R12 pad 1: Net-(U2A--) -> Net-(U2D--)
- R12 pad 2: /Analog/AmpCathode -> Net-(R12-Pad2)
- R13 pad 1: Net-(D3-K) -> Net-(U2A--)
- R13 pad 2: /Analog/Env -> /Analog/AmpCathode
- R14 pad 1: Net-(R11-Pad2) -> /Analog/Env
- R14 pad 2: /Analog/SumPt -> Net-(R14-Pad2)
- R15 pad 1: /Analog/Env -> Net-(R12-Pad2)
- R15 pad 2: Net-(R15-Pad2) -> /Analog/SumPt
- R18 pad 2: Net-(U2D--) -> Net-(U2B--)
- R2 pad 1: CLOSED_OUT -> Net-(U1B-+)
- R2 pad 2: Net-(Q1-B) -> GND
- R20 pad 1: Net-(U2D--) -> Net-(R20-Pad1)
- R20 pad 2: /Analog/AmpAnode -> OPEN_IN
- R21 pad 1: Net-(U2C--) -> Net-(U2B--)
- R21 pad 2: Net-(C11-Pad1) -> /Analog/AmpAnode
- R22 pad 1: Net-(R22-Pad1) -> Net-(U2C--)
- R22 pad 2: OPEN_IN -> Net-(C10-Pad1)
- R24 pad 1: Net-(C13-Pad2) -> Net-(C11-Pad2)
- R24 pad 2: Net-(U3A--) -> +9V
- R25 pad 1: Net-(U3A--) -> GND
- R25 pad 2: Net-(R25-Pad2) -> Net-(C11-Pad2)
- R26 pad 1: Net-(R25-Pad2) -> Net-(C11-Pad2)
- R26 pad 2: Net-(U3B--) -> Net-(U1C--)
- R3 pad 1: Net-(D1-A) -> CLOSED_OUT
- R3 pad 2: /Analog/HalfRect -> Net-(Q1-B)
- R4 pad 1: +9V -> Net-(C5-Pad2)
- R4 pad 2: Net-(Q1-C) -> Net-(D2-A)
- R5 pad 1: /Analog/HalfRect -> +9V
- R5 pad 2: Net-(U1D-+) -> Net-(D1-A)
- R6 pad 1: +9V -> Net-(D2-A)
- R6 pad 2: Net-(Q2-C) -> /Analog/HalfRect
- R7 pad 1: +9V -> Net-(D1-K)
- R7 pad 2: Net-(U1B-+) -> Net-(R10-Pad1)
- R8 pad 1: Net-(U1B-+) -> Net-(C6-Pad2)
- R8 pad 2: GND -> Net-(U2D--)
- R9 pad 1: Net-(C7-Pad2) -> Net-(R10-Pad1)
- R9 pad 2: Net-(U2B--) -> /Analog/VG
- RV1 pad 1: Net-(R15-Pad2) -> Net-(R14-Pad2)
- TP3 pad 1: /Analog/Thresh -> /Analog/Env
- TP7 pad 1: LOOP_OUT -> TUNE_IN
- U1 pad 1: Net-(D1-K) -> Net-(D2-K)
- U1 pad 10: /Analog/Env -> /Analog/VG
- U1 pad 12: Net-(U1D-+) -> /Analog/Env
- U1 pad 13: /Analog/Env -> /Analog/Thresh
- U1 pad 14: Net-(D3-A) -> Net-(R20-Pad1)
- U1 pad 2: Net-(D1-A) -> Net-(D2-A)
- U1 pad 8: Net-(R22-Pad1) -> Net-(R27-Pad1)
- U1 pad 9: /Analog/Thresh -> Net-(U1C--)
- U2 pad 14: /Analog/AmpAnode -> Net-(R12-Pad2)
- U2 pad 7: Net-(R11-Pad2) -> /Analog/AmpAnode
- U2 pad 8: Net-(C11-Pad1) -> Net-(C10-Pad1)
- U3 pad 1: Net-(R25-Pad2) -> /Digital/SDA
- U3 pad 2: Net-(U3A--) -> unconnected-(U3-PC14/PB9-Pad2)
- U3 pad 3: /Analog/VG -> unconnected-(U3-PC15-Pad3)
- U3 pad 4: GND -> +3.3V
- U3 pad 5: /Analog/VG -> GND
- U3 pad 6: Net-(U3B--) -> NRST
- U3 pad 7: Net-(R27-Pad1) -> unconnected-(U3-PA0-Pad7)
- U3 pad 8: +9V -> /Digital/TunerModeIn
- U4 pad 1: /Digital/SDA -> GND
- U4 pad 2: unconnected-(U4-PC14/PB9-Pad2) -> +3.3V
- U4 pad 3: unconnected-(U4-PC15-Pad3) -> +9V
- U5 pad 3: +9V -> /Digital/SCL
Other:
- board size 55.7 x 44.8 mm -> 55.6 x 45.5 mm
- board text removed: "A"
- board text removed: "B"
- board text removed: "FX_IN"
- board text removed: "FX_OUT"
- board text removed: "GND"
- board text removed: "L_IN"
- board text removed: "L_OUT"
- board text removed: "NRST"
- board text removed: "SWCLK"
- board text removed: "SWDIO"
- board text removed: "VCC"

Commit message: routed, DRC passing
Parts:
- moved J1 0.90 mm to (52.3, 12.9)
Connections:
- J4 pad 1: FX_OUT -> FX_IN
- J4 pad 2: FX_IN -> FX_OUT
Routing:
- net +9V: track 0.00 -> 123.0 mm, vias 0 -> 5
- net /Analog/VG: track 0.00 -> 85.3 mm, vias 0 -> 3
- net +3.3V: track 0.00 -> 83.5 mm, vias 0 -> 4
- net FX_IN: track 0.00 -> 66.0 mm, vias 0 -> 2
- net /Digital/GateByp: track 0.00 -> 39.8 mm, vias 0 -> 1
- net CLOSED_OUT: track 0.00 -> 37.9 mm, vias 0 -> 1
- net GND: track 0.00 -> 37.7 mm, vias 0 -> 22
- net /Digital/TunerModeIn: track 0.00 -> 37.5 mm
- net NRST: track 0.00 -> 31.5 mm, vias 0 -> 1
- net /Analog/AmpCathode: track 0.00 -> 30.8 mm
- net /Digital/GateLED: track 0.00 -> 30.3 mm, vias 0 -> 2
- net /Analog/Thresh: track 0.00 -> 28.5 mm, vias 0 -> 2
- net OPEN_IN: track 0.00 -> 26.5 mm, vias 0 -> 1
- net /Analog/SumPt: track 0.00 -> 20.5 mm, vias 0 -> 2
- net SWDIO: track 0.00 -> 20.5 mm
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
Commit message: silkscreen and tweaks
Parts:
- moved J5 0.40 mm to (18.9, 6.38)
Routing:
- net /Analog/SumPt: track 20.5 -> 21.2 mm
- net GND: vias 22 -> 24
Other:
- board text added: "CLK"
- board text added: "DIO"
- board text added: "FI"
- board text added: "FO"
- board text added: "GND"
- board text added: "Handyman v2"
- board text added: "LI"
- board text added: "LO"
- board text added: "NRST"
- board text added: "Rev2 July 2025 Hayden Setlik"
- board text added: "VCC"
