File: AttenuatorSim/AttenuatorSim.kicad_sch (KiCad schematic)
At the start: 28 parts, among them Q1 BC847, U1 TL074

Commit message: tweaks to analog circuit
Parts:
- added C2: 47n, symbol Device:C
- C3: value 1u -> 100n
- R3, R6: value 47k -> 33k
Connections:
- net VG: now also C2.2
- net at R3.2, R5.1, R6.1: now also C2.1
Other:
- moved on the sheet: R5
Changed lines of the file:
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@@
 	)
 	(junction
+		(at 118.11 80.645)
+		(diameter 0)
+		(color 0 0 0 0)
+	)
+	(junction
 		(at 78.74 102.87)
 		(diameter 0)
@@
 	)
 	(junction
+		(at 118.11 67.31)
+		(diameter 0)
+		(color 0 0 0 0)
+	)
+	(junction
 		(at 120.65 96.52)
 		(diameter 0)
@@
 	(wire
 		(pts
+			(xy 107.95 70.485) (xy 107.95 67.31)
+		)
+		(stroke
+			(width 0)
+			(type default)
+		)
+	)
+	(wire
+		(pts
 			(xy 78.74 100.33) (xy 78.74 102.87)
 		)
@@
 	(wire
 		(pts
+			(xy 118.11 67.31) (xy 118.11 70.485)
+		)
+		(stroke
+			(width 0)
+			(type default)
+		)
+	)
+	(wire
+		(pts
 			(xy 73.66 102.87) (xy 78.74 102.87)
 		)
@@
 	(wire
 		(pts
+			(xy 118.11 80.645) (xy 118.11 83.82)
+		)
+		(stroke
+			(width 0)
+			(type default)
+		)
+	)
+	(wire
+		(pts
 			(xy 190.5 69.85) (xy 219.71 69.85)
 		)
@@
 	(wire
 		(pts
+			(xy 107.95 67.31) (xy 118.11 67.31)
+		)
+		(stroke
+			(width 0)
+			(type default)
+		)
+	)
+	(wire
+		(pts
 			(xy 118.11 64.77) (xy 120.65 64.77)
 		)
@@
 	(wire
 		(pts
+			(xy 107.95 78.105) (xy 107.95 80.645)
+		)
+		(stroke
+			(width 0)
+			(type default)
+		)
+	)
+	(wire
+		(pts
 			(xy 149.86 109.22) (xy 149.86 110.49)
 		)
@@
 	(wire
 		(pts
+			(xy 107.95 80.645) (xy 118.11 80.645)
+		)
+		(stroke
+			(width 0)
+			(type default)
+		)
+	)
+	(wire
+		(pts
 			(xy 168.91 99.06) (xy 171.45 99.06)
 		)
@@
 	(wire
 		(pts
-			(xy 118.11 64.77) (xy 118.11 74.295)
+			(xy 118.11 64.77) (xy 118.11 67.31)
 		)
 		(stroke
@@
 	(wire
 		(pts
-			(xy 118.11 81.915) (xy 118.11 83.82)
+			(xy 118.11 78.105) (xy 118.11 80.645)
 		)
 		(stroke
@@
 			)
 		)
-		(property "Sim.Params" "dc=0 ampl=0.2 f=330 td=0 theta=0 phase=0 ac=1"
+		(property "Sim.Params" "dc=0 ampl=0.4 f=330 td=0 theta=0 phase=0 ac=1"
 			(at 26.67 132.5851 0)
 			(effects
@@
 	)
 	(symbol
+		(lib_id "Device:C")
+		(at 107.95 74.295 0)
+		(unit 1)
+		(exclude_from_sim no)
+		(in_bom yes)
+		(on_board yes)
+		(dnp no)
+		(fields_autoplaced yes)
+		(property "Reference" "C2"
+			(at 111.76 73.0249 0)
+			(effects
+				(font
+					(size 1.27 1.27)
+				)
+				(justify left)
+			)
+		)
+		(property "Value" "47n"
+			(at 111.76 75.5649 0)
+			(effects
+				(font
+					(size 1.27 1.27)
+				)
+				(justify left)
+			)
+		)
+		(property "Footprint" ""
+			(at 108.9152 78.105 0)
+			(effects
+				(font
+					(size 1.27 1.27)
+				)
+				(hide yes)
+			)
+		)
+		(property "Datasheet" "~"
+			(at 107.95 74.295 0)
+			(effects
+				(font
+					(size 1.27 1.27)
+				)
+				(hide yes)
+			)
+		)
+		(property "Description" "Unpolarized capacitor"
+			(at 107.95 74.295 0)
+			(effects
+				(font
+					(size 1.27 1.27)
+				)
+				(hide yes)
+			)
+		)
+		(pin "2"
+		)
+		(pin "1"
+		)
+		(instances
+			(project "AttenuatorSim"
+				(path "/98bc47f1-8090-4985-b644-bda5d553ef6a"
+					(reference "C2")
+					(unit 1)
+				)
+			)
+		)
+	)
+	(symbol
 		(lib_id "Diode:1N4148W")
 		(at 149.86 114.3 270)
@@
 			)
 		)
-		(property "Value" "47k"
+		(property "Value" "33k"
 			(at 124.46 60.96 90)
 			(effects
@@
 			)
 		)
-		(property "Value" "47k"
+		(property "Value" "33k"
 			(at 112.395 60.96 90)
 			(effects
@@
 	(symbol
 		(lib_id "Device:R_US")
-		(at 118.11 78.105 0)
+		(at 118.11 74.295 0)
 		(unit 1)
 		(exclude_from_sim no)
@@
 		(fields_autoplaced yes)
 		(property "Reference" "R5"
-			(at 120.65 76.8349 0)
+			(at 120.65 73.0249 0)
 			(effects
 				(font
@@
 		)
 		(property "Value" "10k"
-			(at 120.65 79.3749 0)
+			(at 120.65 75.5649 0)
 			(effects
 				(font
@@
 		)
 		(property "Footprint" "Resistor_SMD:R_0805_2012Metric"
-			(at 119.126 78.359 90)
+			(at 119.126 74.549 90)
 			(effects
 				(font
@@
 		)
 		(property "Datasheet" "~"
-			(at 118.11 78.105 0)
+			(at 118.11 74.295 0)
 			(effects
 				(font
@@
 		)
 		(property "Description" "Resistor, US symbol"
-			(at 118.11 78.105 0)
+			(at 118.11 74.295 0)
 			(effects
 				(font
@@
 			)
 		)
-		(property "Value" "1u"
+		(property "Value" "100n"
 			(at 104.14 91.44 90)
 			(effects

Commit message: new prelim routing, DRC passing
Parts:
- removed V3: 4.5, symbol Simulation_SPICE:VDC
- added C6: 100n, Capacitor_SMD:C_0805_2012Metric, symbol Device:C
- added R14, R15: 47k, Resistor_SMD:R_0805_2012Metric, symbol Device:R_US
- added U2: TL074, symbol Amplifier_Operational:TL074
Connections:
- net +9V: now also C6.1, R14.1, U2.4 (V+)
- net 0: now also C6.2, R15.2, U2.11 (V-)
- net VG: now also U2.6 (-), U2.7
- new net: R14.2, R15.1, U2.5 (+)
