File: Simulations/Attenuator/Attenuator.kicad_sch (KiCad schematic)
At the start: 27 parts, among them Q1 BC847, U1 TL074

Commit message: noise schematic tweaks
Parts:
- added R15, R16: 220, Resistor_SMD:R_0805_2012Metric, symbol Device:R_US
- C11: value 47n -> 10n
- V2: value 0 -> ${SIM.PARAMS}
Connections:
- net AmpAnode: now also R16.2; no longer D5.2 (A)
- net AmpCathode: now also R15.1; no longer D2.1 (K)
- net Vgate: now reaches R1.1, V2.1
- new net: D2.1 (K), R15.2
- new net: D5.2 (A), R16.1
Changed lines of the file:
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@@
 	(wire
 		(pts
+			(xy 144.78 76.2) (xy 144.78 77.47)
+		)
+		(stroke
+			(width 0)
+			(type default)
+		)
+	)
+	(wire
+		(pts
 			(xy 113.03 63.5) (xy 113.03 66.04)
 		)
@@
 	(wire
 		(pts
-			(xy 214.63 116.84) (xy 144.78 116.84)
+			(xy 214.63 137.16) (xy 144.78 137.16)
 		)
 		(stroke
@@
 	(wire
 		(pts
-			(xy 144.78 66.04) (xy 144.78 77.47)
+			(xy 144.78 66.04) (xy 144.78 68.58)
 		)
 		(stroke
@@
 	(wire
 		(pts
+			(xy 144.78 121.92) (xy 144.78 116.84)
+		)
+		(stroke
+			(width 0)
+			(type default)
+		)
+	)
+	(wire
+		(pts
 			(xy 134.62 87.63) (xy 134.62 97.79)
 		)
@@
 	(wire
 		(pts
-			(xy 214.63 68.58) (xy 214.63 116.84)
+			(xy 214.63 68.58) (xy 214.63 137.16)
 		)
 		(stroke
@@
 	(wire
 		(pts
+			(xy 144.78 137.16) (xy 144.78 129.54)
+		)
+		(stroke
+			(width 0)
+			(type default)
+		)
+	)
+	(wire
+		(pts
 			(xy 125.73 63.5) (xy 127 63.5)
 		)
@@
 	)
 	(label "AmpAnode"
-		(at 157.48 116.84 180)
+		(at 157.48 137.16 180)
 		(effects
 			(font
@@
 		)
 	)
+	(label "Vgate"
+		(at 52.07 68.58 0)
+		(effects
+			(font
+				(size 1.27 1.27)
+			)
+			(justify left bottom)
+		)
+	)
 	(label "Vbase"
 		(at 69.85 68.58 0)
@@
 			)
 		)
-		(property "Value" "47n"
+		(property "Value" "10n"
 			(at 104.775 73.6599 0)
 			(show_name no)
@@
 	)
 	(symbol
+		(lib_id "Device:R_US")
+		(at 144.78 72.39 0)
+		(unit 1)
+		(body_style 1)
+		(exclude_from_sim no)
+		(in_bom yes)
+		(on_board yes)
+		(in_pos_files yes)
+		(dnp no)
+		(fields_autoplaced yes)
+		(property "Reference" "R15"
+			(at 147.32 71.1199 0)
+			(show_name no)
+			(do_not_autoplace no)
+			(effects
+				(font
+					(size 1.27 1.27)
+				)
+				(justify left)
+			)
+		)
+		(property "Value" "220"
+			(at 147.32 73.6599 0)
+			(show_name no)
+			(do_not_autoplace no)
+			(effects
+				(font
+					(size 1.27 1.27)
+				)
+				(justify left)
+			)
+		)
+		(property "Footprint" "Resistor_SMD:R_0805_2012Metric"
+			(at 145.796 72.644 90)
+			(hide yes)
+			(show_name no)
+			(do_not_autoplace no)
+			(effects
+				(font
+					(size 1.27 1.27)
+				)
+			)
+		)
+		(property "Datasheet" ""
+			(at 144.78 72.39 0)
+			(hide yes)
+			(show_name no)
+			(do_not_autoplace no)
+			(effects
+				(font
+					(size 1.27 1.27)
+				)
+			)
+		)
+		(property "Description" "Resistor, US symbol"
+			(at 144.78 72.39 0)
+			(hide yes)
+			(show_name no)
+			(do_not_autoplace no)
+			(effects
+				(font
+					(size 1.27 1.27)
+				)
+			)
+		)
+		(pin "2"
+		)
+		(pin "1"
+		)
+		(instances
+			(project "Attenuator"
+				(path "/896e8929-6be2-4dd7-af77-210e443a477f"
+					(reference "R15")
+					(unit 1)
+				)
+			)
+		)
+	)
+	(symbol
 		(lib_id "Diode:1N4148W")
 		(at 144.78 90.17 90)
@@
 			)
 		)
-		(property "Value" "0"
+		(property "Value" "${SIM.PARAMS}"
 			(at 55.88 77.3401 0)
+			(hide yes)
 			(show_name no)
 			(do_not_autoplace no)
@@
 			)
 		)
-		(property "Sim.Type" "DC"
+		(property "Sim.Type" "PULSE"
 			(at 52.07 76.2 0)
 			(hide yes)
@@
 			)
 		)
+		(property "Sim.Params" "y1=0 y2=3.3 td=85m tr=0 tf=0 tw=50m per=70m np=1"
+			(at 52.07 76.2 0)
+			(hide yes)
+			(show_name no)
+			(do_not_autoplace no)
+			(effects
+				(font
+					(size 1.27 1.27)
+				)
+			)
+		)
 		(pin "1"
 		)
@@
 					(unit 1)
 				)
+			)
+		)
+	)
+	(symbol
+		(lib_id "Device:R_US")
+		(at 144.78 125.73 0)
+		(unit 1)
+		(body_style 1)
+		(exclude_from_sim no)
+		(in_bom yes)
+		(on_board yes)
+		(in_pos_files yes)
+		(dnp no)
+		(fields_autoplaced yes)
+		(property "Reference" "R16"
+			(at 147.32 124.4599 0)
+			(show_name no)
+			(do_not_autoplace no)
+			(effects
+				(font
+					(size 1.27 1.27)
+				)
+				(justify left)
+			)
+		)
+		(property "Value" "220"
+			(at 147.32 126.9999 0)
+			(show_name no)
+			(do_not_autoplace no)
+			(effects
+				(font
+					(size 1.27 1.27)
+				)
+				(justify left)
+			)
+		)
+		(property "Footprint" "Resistor_SMD:R_0805_2012Metric"
+			(at 145.796 125.984 90)
+			(hide yes)
+			(show_name no)
+			(do_not_autoplace no)
+			(effects
+				(font
+					(size 1.27 1.27)
+				)
+			)
+		)
+		(property "Datasheet" ""
+			(at 144.78 125.73 0)
+			(hide yes)
+			(show_name no)
+			(do_not_autoplace no)
+			(effects
+				(font
+					(size 1.27 1.27)
+				)
+			)
+		)
+		(property "Description" "Resistor, US symbol"
+			(at 144.78 125.73 0)
+			(hide yes)
+			(show_name no)
+			(do_not_autoplace no)
+			(effects
+				(font
+					(size 1.27 1.27)
+				)
+			)
+		)
+		(pin "2"
+		)
+		(pin "1"
+		)
+		(instances
+			(project "Attenuator"
+				(path "/896e8929-6be2-4dd7-af77-210e443a477f"
+					(reference "R16")
+					(unit 1)
+				)

Commit message: switched to FET controlled gate circuit
Parts:
- removed Q1: BC847, Package_TO_SOT_SMD:SOT-23, symbol Transistor_BJT:BC847
- removed R1: 10k, Resistor_SMD:R_0805_2012Metric, symbol Device:R_US
- added Q2: NMOS, symbol Simulation_SPICE:NMOS
Connections:
- net Vgate is gone; now on net Vbase: V2.1
- net GND: now also Q2.3 (S)
- net Vbase: now also Q2.2 (G)
- net Vfet: now reaches D1.2 (A), R2.2
- net Vfet: now also Q2.1 (D)
Other:
- moved on the sheet: C1, C11, C12, D1, D2, D3, D4, D5, R10, R11, R12, R13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
